File: discipline-pcb.kicad_pcb (KiCad board)
At the start: 2 copper layers, 304.9 x 122.8 mm, 180 parts, among them J1 AVR-ISP-6, SW1 KEYSW, SW10 KEYSW, SW11 KEYSW, SW12 KEYSW, SW13 KEYSW, SW14 KEYSW, SW15 KEYSW, SW16 KEYSW, SW17 KEYSW, SW18 KEYSW, SW19 KEYSW, SW2 KEYSW, SW20 KEYSW, SW21 KEYSW, SW22 KEYSW, SW23 KEYSW, SW24 KEYSW, SW25 KEYSW, SW26 KEYSW, SW27 KEYSW, SW28 KEYSW, SW29 KEYSW, SW3 KEYSW, SW30 KEYSW, SW31 KEYSW, SW32 KEYSW, SW33 KEYSW, SW34 KEYSW, SW35 KEYSW, SW36 KEYSW, SW37 KEYSW, SW38 KEYSW, SW39 KEYSW, SW4 KEYSW, SW40 KEYSW, SW41 KEYSW, SW42 KEYSW, SW43 KEYSW, SW44 KEYSW, SW45 KEYSW, SW46 KEYSW, SW47 KEYSW, SW48 KEYSW, SW49 KEYSW, SW5 KEYSW, SW50 KEYSW, SW51 KEYSW, SW52 KEYSW, SW53 KEYSW, SW54 KEYSW, SW55 KEYSW, SW56 KEYSW, SW57 KEYSW, SW58 KEYSW, SW59 KEYSW, SW6 KEYSW, SW60 KEYSW, SW61 KEYSW, SW62 KEYSW, SW63 KEYSW, SW64 KEYSW, SW65 KEYSW, SW66 KEYSW, SW67 KEYSW, SW68 KEYSW, SW69 KEYSW, SW7 KEYSW, SW70 KEYSW, SW71 KEYSW, SW72 KEYSW, SW73 KEYSW, SW74 KEYSW, SW8 KEYSW, SW9 KEYSW, U1 ATmega32A-PU, Y1 Crystal

Commit message: added numpad to pcb, still need layout updates
Parts:
- removed G*** (x2): LOGO, logos:TOPY 4MM MASK
- removed G***: LOGO, logos:DISCIPLINE_SMALL_MASK
- removed G***: LOGO, logos:DISCIPLINE_SMALL_COPPER
- removed REF**: 6.25U, cftkb:MX-6.25U-Stabilizer
- removed REF** (x10): MountingHole_2.2mm_M2_Pad, MountingHole:MountingHole_2.2mm_M2_Pad
- removed ST72: 7U, cftkb:MX-7U-Stabilizer
- added D75: , cftkb:D_DO-35_SOD27_P5.08mm_Horizontal, F.Cu at (351.3, 66.5)
- added D76: , cftkb:D_DO-35_SOD27_P5.08mm_Horizontal, F.Cu at (364.3, 66.5)
- added D77: , cftkb:D_DO-35_SOD27_P5.08mm_Horizontal, F.Cu at (377.2, 66.5)
- added D78: , cftkb:D_DO-35_SOD27_P5.08mm_Horizontal, F.Cu at (354.9, 68.1)
- added D79: , cftkb:D_DO-35_SOD27_P5.08mm_Horizontal, F.Cu at (367.4, 68.1)
- added D80: , cftkb:D_DO-35_SOD27_P5.08mm_Horizontal, F.Cu at (380.5, 68.1)
- added D81: , cftkb:D_DO-35_SOD27_P5.08mm_Horizontal, F.Cu at (357.9, 69.8)
- added D82: , cftkb:D_DO-35_SOD27_P5.08mm_Horizontal, F.Cu at (370.6, 69.8)
- added D83: , cftkb:D_DO-35_SOD27_P5.08mm_Horizontal, F.Cu at (361.0, 71.4)
- added D84: , cftkb:D_DO-35_SOD27_P5.08mm_Horizontal, F.Cu at (373.7, 71.4)
- added D85: , cftkb:D_DO-35_SOD27_P5.08mm_Horizontal, F.Cu at (383.6, 69.8)
- added D86: , cftkb:D_DO-35_SOD27_P5.08mm_Horizontal, F.Cu at (390.4, 66.5)
- added D87: , cftkb:D_DO-35_SOD27_P5.08mm_Horizontal, F.Cu at (386.9, 71.4)
- added SW75: KEYSW, cftkb:SW_Cherry_MX1A_1.00u_PCB-NOSCREEN, F.Cu at (380.2, 89.7)
- added SW76: KEYSW, cftkb:SW_Cherry_MX1A_1.00u_PCB-NOSCREEN, F.Cu at (399.3, 89.7)
- added SW77: KEYSW, cftkb:SW_Cherry_MX1A_1.00u_PCB-NOSCREEN, F.Cu at (418.3, 89.7)
- added SW78: KEYSW, cftkb:SW_Cherry_MX1A_1.00u_PCB-NOSCREEN, F.Cu at (380.2, 108.7)
- added SW79: KEYSW, cftkb:SW_Cherry_MX1A_1.00u_PCB-NOSCREEN, F.Cu at (399.3, 108.7)
- added SW80: KEYSW, cftkb:SW_Cherry_MX1A_2.00u_PCBNOSCREEN, F.Cu at (420.8, 125.9)
- added SW81: KEYSW, cftkb:SW_Cherry_MX1A_1.00u_PCB-NOSCREEN, F.Cu at (380.3, 127.8)
- added SW82: KEYSW, cftkb:SW_Cherry_MX1A_1.00u_PCB-NOSCREEN, F.Cu at (399.3, 127.8)
- added SW83: KEYSW, cftkb:SW_Cherry_MX1A_1.00u_PCB-NOSCREEN, F.Cu at (380.2, 146.8)
- added SW84: KEYSW, cftkb:SW_Cherry_MX1A_1.00u_PCB-NOSCREEN, F.Cu at (399.3, 146.8)
- added SW85: KEYSW, cftkb:SW_Cherry_MX1A_2.00u_PCBNOSCREEN, F.Cu at (420.8, 164.0)
- added SW86: KEYSW, cftkb:SW_Cherry_MX1A_1.00u_PCB-NOSCREEN, F.Cu at (380.2, 165.9)
- added SW87: KEYSW, cftkb:SW_Cherry_MX1A_1.00u_PCB-NOSCREEN, F.Cu at (399.3, 165.9)
- C4, C5: footprint cftkb:C_Disc_D4.3mm_W1.9mm_P5.00mm -> cftkb:D_DO-35_SOD27_P5.08mm_Horizontal
- SW63, SW64: footprint cftkb:SW_Cherry_MX1A_1.00u_PCB-NOSCREEN -> cftkb:SW_Cherry_MX1A_1.25u_PCBNOSCREEN
- moved SW15 9.52 mm to (361.2, 89.7)
- moved SW30 9.52 mm to (361.2, 108.7)
- moved SW44 9.52 mm to (361.2, 127.8)
- moved SW58 9.52 mm to (361.2, 146.8)
- moved SW57 6.74 mm to (337.3, 151.6)
- moved SW65 6.74 mm to (318.3, 170.7)
- moved SW66 6.74 mm to (337.3, 170.7)
- moved SW67 6.74 mm to (356.4, 170.7)
Other:
- board size 304.9 x 122.8 mm -> 371.6 x 454.1 mm
