File: discipline-pcb.kicad_pcb (KiCad board)
At the start: 2 copper layers, 371.6 x 454.1 mm, 190 parts, among them J1 AVR-ISP-6, SW1 KEYSW, SW10 KEYSW, SW11 KEYSW, SW12 KEYSW, SW13 KEYSW, SW14 KEYSW, SW15 KEYSW, SW16 KEYSW, SW17 KEYSW, SW18 KEYSW, SW19 KEYSW, SW2 KEYSW, SW20 KEYSW, SW21 KEYSW, SW22 KEYSW, SW23 KEYSW, SW24 KEYSW, SW25 KEYSW, SW26 KEYSW, SW27 KEYSW, SW28 KEYSW, SW29 KEYSW, SW3 KEYSW, SW30 KEYSW, SW31 KEYSW, SW32 KEYSW, SW33 KEYSW, SW34 KEYSW, SW35 KEYSW, SW36 KEYSW, SW37 KEYSW, SW38 KEYSW, SW39 KEYSW, SW4 KEYSW, SW40 KEYSW, SW41 KEYSW, SW42 KEYSW, SW43 KEYSW, SW44 KEYSW, SW45 KEYSW, SW46 KEYSW, SW47 KEYSW, SW48 KEYSW, SW49 KEYSW, SW5 KEYSW, SW50 KEYSW, SW51 KEYSW, SW52 KEYSW, SW53 KEYSW, SW54 KEYSW, SW55 KEYSW, SW56 KEYSW, SW57 KEYSW, SW58 KEYSW, SW59 KEYSW, SW6 KEYSW, SW60 KEYSW, SW61 KEYSW, SW62 KEYSW, SW63 KEYSW, SW64 KEYSW, SW65 KEYSW, SW66 KEYSW, SW67 KEYSW, SW68 KEYSW, SW69 KEYSW, SW7 KEYSW, SW70 KEYSW, SW71 KEYSW, SW72 KEYSW, SW73 KEYSW, SW74 KEYSW, SW75 KEYSW, SW76 KEYSW, SW77 KEYSW, SW78 KEYSW, SW79 KEYSW, SW8 KEYSW, SW80 KEYSW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

Commit message: EOD
Routing:
- net Net-(D65-Pad2): track 215.1 -> 182.3 mm
- net Net-(D58-Pad2): track 142.1 -> 153.5 mm
- net Net-(D44-Pad2): track 119.9 -> 129.4 mm
- net Net-(D15-Pad2): track 78.0 -> 87.5 mm
- net Net-(D30-Pad2): track 96.9 -> 106.4 mm
- net Net-(D67-Pad2): track 163.1 -> 170.0 mm
- net Net-(D57-Pad2): track 151.1 -> 157.8 mm
- net Net-(D66-Pad2): track 190.5 -> 187.6 mm
Other:
- board size 371.6 x 454.1 mm -> 371.6 x 127.6 mm
