File: NumDiscipline-pcb.kicad_pcb (KiCad board)
At the start: 2 copper layers, 371.6 x 127.6 mm, 190 parts, among them J1 AVR-ISP-6, SW1 KEYSW, SW10 KEYSW, SW11 KEYSW, SW12 KEYSW, SW13 KEYSW, SW14 KEYSW, SW15 KEYSW, SW16 KEYSW, SW17 KEYSW, SW18 KEYSW, SW19 KEYSW, SW2 KEYSW, SW20 KEYSW, SW21 KEYSW, SW22 KEYSW, SW23 KEYSW, SW24 KEYSW, SW25 KEYSW, SW26 KEYSW, SW27 KEYSW, SW28 KEYSW, SW29 KEYSW, SW3 KEYSW, SW30 KEYSW, SW31 KEYSW, SW32 KEYSW, SW33 KEYSW, SW34 KEYSW, SW35 KEYSW, SW36 KEYSW, SW37 KEYSW, SW38 KEYSW, SW39 KEYSW, SW4 KEYSW, SW40 KEYSW, SW41 KEYSW, SW42 KEYSW, SW43 KEYSW, SW44 KEYSW, SW45 KEYSW, SW46 KEYSW, SW47 KEYSW, SW48 KEYSW, SW49 KEYSW, SW5 KEYSW, SW50 KEYSW, SW51 KEYSW, SW52 KEYSW, SW53 KEYSW, SW54 KEYSW, SW55 KEYSW, SW56 KEYSW, SW57 KEYSW, SW58 KEYSW, SW59 KEYSW, SW6 KEYSW, SW60 KEYSW, SW61 KEYSW, SW62 KEYSW, SW63 KEYSW, SW64 KEYSW, SW65 KEYSW, SW66 KEYSW, SW67 KEYSW, SW68 KEYSW, SW69 KEYSW, SW7 KEYSW, SW70 KEYSW, SW71 KEYSW, SW72 KEYSW, SW73 KEYSW, SW74 KEYSW, SW75 KEYSW, SW76 KEYSW, SW77 KEYSW, SW78 KEYSW, SW79 KEYSW, SW8 KEYSW, SW80 KEYSW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

Commit message: new routing fixed, ready for checkover
Parts:
- added G***: LOGO, cftkb:NumDiscipline_SMALL_COPPER, F.Cu at (152.9, 164.5)
- added REF**: MountingHole_2.2mm_M2_Pad, cftkb:MountingHole_2.2mm_M2_Pad, F.Cu at (242.4, 78.9)
- added REF**: MountingHole_2.2mm_M2_Pad, cftkb:MountingHole_2.2mm_M2_Pad, F.Cu at (58.6, 80.5)
- added REF**: MountingHole_2.2mm_M2_Pad, cftkb:MountingHole_2.2mm_M2_Pad, F.Cu at (58.6, 61.4)
- added REF**: MountingHole_2.2mm_M2_Pad, cftkb:MountingHole_2.2mm_M2_Pad, F.Cu at (420.5, 61.4)
- added REF**: MountingHole_2.2mm_M2_Pad, cftkb:MountingHole_2.2mm_M2_Pad, F.Cu at (420.5, 80.5)
- added REF**: MountingHole_2.2mm_M2_Pad, cftkb:MountingHole_2.2mm_M2_Pad, F.Cu at (96.4, 161.4)
- added REF**: MountingHole_2.2mm_M2_Pad, cftkb:MountingHole_2.2mm_M2_Pad, F.Cu at (205.6, 161.4)
- added REF**: MountingHole_2.2mm_M2_Pad, cftkb:MountingHole_2.2mm_M2_Pad, F.Cu at (314.8, 161.4)
- added REF**: MountingHole_2.2mm_M2_Pad, cftkb:MountingHole_2.2mm_M2_Pad, F.Cu at (365.6, 161.4)
- added REF**: MountingHole_2.2mm_M2_Pad, cftkb:MountingHole_2.2mm_M2_Pad, F.Cu at (365.6, 104.3)
- added REF**: MountingHole_2.2mm_M2_Pad, cftkb:MountingHole_2.2mm_M2_Pad, F.Cu at (298.3, 104.3)
- added REF**: MountingHole_2.2mm_M2_Pad, cftkb:MountingHole_2.2mm_M2_Pad, F.Cu at (206.2, 104.3)
- added REF**: MountingHole_2.2mm_M2_Pad, cftkb:MountingHole_2.2mm_M2_Pad, F.Cu at (111.0, 104.3)
- moved C5 1.24 mm to (319.2, 78.7)
Routing:
- net Net-(D63-Pad2): track 0.00 -> 605.3 mm
- net col17: track 75.3 -> 226.5 mm, vias 0 -> 4
- net col15: track 57.2 -> 202.0 mm, vias 0 -> 4
- net col16: track 76.2 -> 186.6 mm, vias 0 -> 4
- net row4: track 328.1 -> 402.3 mm, vias 0 -> 2
- net row2: track 269.4 -> 338.5 mm, vias 2 -> 3
- net row3: track 314.7 -> 380.7 mm, vias 3 -> 4
- net row0: track 292.3 -> 351.2 mm, vias 1 -> 2
- net row1: track 297.1 -> 354.7 mm, vias 2 -> 3
- net GND: track 214.9 -> 245.4 mm, vias 1 -> 17
- net boot: track 120.6 -> 126.3 mm
- net Net-(D77-Pad2): track 42.6 -> 38.3 mm
- net col2: track 329.2 -> 333.2 mm
- net +5V: track 147.9 -> 151.9 mm
- net col12: track 191.1 -> 194.1 mm
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- added copper zone on B.Cu, net GND
Other:
- board text added: "#"
- board text added: "#DISCIPLINE - 65% keyboard + Numpad - (del, page up/down, insert)"
- board text added: "Revised lauer2356 27April2020"
- board text added: "coseyfannitutti 2019 - rev1 lauer2356 2020 - rev 2.1 (numpad)"
- board text removed: "7/2/2019"
- board text removed: "DISCIPLINE - 65% keyboard made with only through hole components"
- board text removed: "coseyfannitutti 2019 rev1"

Commit message: add plate
Parts:
- removed G***: LOGO, cftkb:NumDiscipline_SMALL_COPPER
- added REF**: NumDiscipline_SMALL_COPPER, cftkb:NumDiscipline_SMALL_COPPER, F.Cu at (152.9, 164.5)
- added REF**: NumDiscipline_SMALL_MASK, cftkb:NumDiscipline_SMALL_MASK, F.Cu at (152.9, 164.5)
- SW1: value KEYSW -> ESCAPE
- SW2: value KEYSW -> 1
Routing:
- net GND: track 245.4 -> 217.4 mm, vias 17 -> 14
- net Net-(D63-Pad2): track 605.3 -> 596.2 mm
- net Net-(D68-Pad2): track 251.3 -> 246.8 mm
- net Net-(D62-Pad2): track 356.3 -> 354.8 mm
- net Net-(D58-Pad2): track 148.7 -> 149.3 mm

Commit message: add 3d, finish plate
Parts:
- removed the REF** at (111.0, 104.3)
- removed the REF** at (205.6, 161.4)
- removed the REF** at (365.6, 161.4)
- removed the REF** at (365.6, 104.3)
- added REF**: NumDiscipline_LARGE_B_SILK, cftkb:NumDiscipline_LARGE_B_SILK, F.Cu at (244.3, 123.3)
- added REF**: MountingHole_2.2mm_M2_Pad, cftkb:MountingHole_2.2mm_M2_Pad, F.Cu at (113.3, 104.3)
- added REF**: MountingHole_2.2mm_M2_Pad, cftkb:MountingHole_2.2mm_M2_Pad, F.Cu at (205.6, 168.6)
- added REF**: MountingHole_2.2mm_M2_Pad, cftkb:MountingHole_2.2mm_M2_Pad, F.Cu at (387.2, 161.4)
- added REF**: MountingHole_2.2mm_M2_Pad, cftkb:MountingHole_2.2mm_M2_Pad, F.Cu at (387.2, 104.3)
- moved REF** 0.79 mm to (299.1, 104.3)
Changed lines of the file:
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@@
     (tracks 2382)
     (zones 0)
-    (modules 205)
+    (modules 206)
     (nets 128)
   )
@@
     (solder_mask_min_width 0.25)
     (aux_axis_origin 0 0)
-    (grid_origin 152.876 164.49675)
+    (grid_origin 420.52875 61.43625)
     (visible_elements 7FFFFFFF)
     (pcbplotparams
@@
     (add_net row4)
   )
+  (module cftkb:NumDiscipline_LARGE_B_SILK (layer F.Cu)
+    (at 244.31625 123.34875)
+    (fp_text reference REF** (at 0 5.08) (layer Cmts.User) hide
+      (effects (font (size 1 1) (thickness 0.15)))
+    )
+    (fp_text value NumDiscipline_LARGE_B_SILK (at 0 -0.5) (layer F.Fab)
+      (effects (font (size 1 1) (thickness 0.15)))
+    )
+    (fp_line (start -53.34 15.24) (end 55.88 15.24) (layer B.SilkS) (width 1))
+    (fp_line (start 55.88 -15.24) (end -53.34 -15.24) (layer B.SilkS) (width 1))
+    (fp_arc (start -53.34 0) (end -53.34 -15.24) (angle -180) (layer B.SilkS) (width 1))
+    (fp_arc (start 55.88 0) (end 55.88 15.24) (angle -180) (layer B.SilkS) (width 1))
+    (fp_text user "#Discipline" (at 0 0) (layer B.SilkS)
+      (effects (font (size 15 15) (thickness 2.5)) (justify mirror))
+    )
+  )
   (module cftkb:NumDiscipline_SMALL_COPPER (layer F.Cu)
     (at 152.876 164.49675)
@@
   )
   (module cftkb:MountingHole_2.2mm_M2_Pad (layer F.Cu)
-    (at 205.58125 161.44875)
+    (at 205.58125 168.5925)
     (descr "Mounting Hole 2.2mm, M2")
     (tags "mounting hole 2.2mm m2")
@@
   )
   (module cftkb:MountingHole_2.2mm_M2_Pad (layer F.Cu)
-    (at 365.60125 161.44875)
+    (at 387.19125 161.44875)
     (descr "Mounting Hole 2.2mm, M2")
     (tags "mounting hole 2.2mm m2")
@@
   )
   (module cftkb:MountingHole_2.2mm_M2_Pad (layer F.Cu)
-    (at 365.60125 104.29875)
+    (at 387.19125 104.29875)
     (descr "Mounting Hole 2.2mm, M2")
     (tags "mounting hole 2.2mm m2")
@@
   )
   (module cftkb:MountingHole_2.2mm_M2_Pad (layer F.Cu)
-    (at 298.29125 104.29875)
+    (at 299.085 104.29875)
     (descr "Mounting Hole 2.2mm, M2")
     (tags "mounting hole 2.2mm m2")
@@
   )
   (module cftkb:MountingHole_2.2mm_M2_Pad (layer F.Cu)
-    (at 110.96625 104.29875)
-    (descr "Mounting Hole 2.2mm, M2")
-    (tags "mounting hole 2.2mm m2")
+    (at 113.3475 104.29875)
+    (descr "Mounting Hole 2.2mm, M2")
+    (tags "mounting hole 2.2mm m2")

Commit message: cleanup files, update readme, add gerbers
Parts:
- added REF**: NumDiscipline_SMALL_FSILK, cftkb:NumDiscipline_SMALL_FSILK, F.Cu at (313.5, 77.3)
- moved RESET1 186.8 mm to (413.2, 62.0), turned to 270 degrees
- moved BOOT1 175.3 mm to (413.2, 74.0), turned to 270 degrees
- moved J1 168.0 mm to (420.5, 71.0), turned to 270 degrees
- moved D87 103.0 mm to (293.0, 59.7)
- moved D86 90.0 mm to (279.0, 66.3)
- moved D84 87.4 mm to (295.5, 59.7)
- moved D85 85.5 mm to (306.8, 62.6)
- moved D83 84.6 mm to (281.7, 66.2)
- moved D82 81.2 mm to (298.3, 61.0)
- moved D80 79.5 mm to (309.6, 63.7)
- moved D81 78.6 mm to (284.4, 67.7)
- moved D79 75.0 mm to (301.1, 62.5)
- moved D77 73.3 mm to (312.4, 65.2)
- moved D78 72.8 mm to (287.2, 69.2)
- moved D76 68.9 mm to (303.9, 64.0)
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Routing:
- net GND: track 217.4 -> 62.8 mm, vias 14 -> 15
- net col14: track 349.4 -> 210.3 mm
- net Net-(D63-Pad2): track 596.2 -> 465.0 mm
- net boot: track 126.3 -> 21.6 mm, vias 2 -> 0
- net Net-(D84-Pad2): track 77.8 -> 168.1 mm
- net Net-(D85-Pad2): track 97.7 -> 184.9 mm
- net Net-(D87-Pad2): track 102.1 -> 188.8 mm
- net Net-(D82-Pad2): track 62.9 -> 145.5 mm
- net Net-(D86-Pad2): track 91.9 -> 174.0 mm
- net Net-(D80-Pad2): track 63.7 -> 143.1 mm
- net Net-(D83-Pad2): track 81.4 -> 154.8 mm
- net Net-(D79-Pad2): track 48.1 -> 120.9 mm
- net Net-(D77-Pad2): track 38.3 -> 109.0 mm
- net Net-(D81-Pad2): track 63.2 -> 132.2 mm
- net Net-(D76-Pad2): track 35.8 -> 102.1 mm
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Other:
- board text removed: "#"
- board text removed: "500mA"
- board text removed: "ISP"

Commit message: start making adjustments from first proto
Parts:
- removed the REF** at (205.6, 168.6)
- added REF**: MountingHole_2.2mm_M2_Pad, cftkb:MountingHole_2.2mm_M2_Pad, F.Cu at (387.2, 92.4)
- added REF**: MountingHole_2.2mm_M2_Pad, cftkb:MountingHole_2.2mm_M2_Pad, F.Cu at (301.5, 92.4)
- added REF**: MountingHole_2.2mm_M2_Pad, cftkb:MountingHole_2.2mm_M2_Pad, F.Cu at (206.2, 94.8)
- added REF**: MountingHole_2.2mm_M2_Pad, cftkb:MountingHole_2.2mm_M2_Pad, F.Cu at (91.9, 92.4)
- added REF**: MountingHole_2.2mm_M2_Pad, cftkb:MountingHole_2.2mm_M2_Pad, F.Cu at (242.4, 61.4)
- added REF**: MountingHole_2.2mm_M2_Pad, cftkb:MountingHole_2.2mm_M2_Pad, F.Cu at (206.1, 171.0)
- added REF**: 6.25U, cftkb:MX-6.25U-Stabilizer, F.Cu at (184.8, 171.0)
- added ST62: 7U, cftkb:MX-7U-Stabilizer, F.Cu at (177.6, 171.0)
- C4, C5: footprint cftkb:D_DO-35_SOD27_P5.08mm_Horizontal -> cftkb:C_Disc_D4.3mm_W1.9mm_P5.00mm
- moved REF** 21.4 mm to (91.9, 104.3)
- moved REF** 4.06 mm to (311.0, 80.5)
- moved F1 2.68 mm to (319.8, 61.8), turned to 180 degrees
- moved REF** 2.38 mm to (301.5, 104.3)
- moved C5 1.35 mm to (373.0, 78.6)
- moved C4 1.27 mm to (377.9, 58.9)
Routing:
- net VCC: track 17.0 -> 22.1 mm
- net Net-(D59-Pad2): track 472.2 -> 475.2 mm
- net +5V: track 210.6 -> 213.2 mm
- net Net-(D79-Pad2): track 120.9 -> 123.1 mm
- net Net-(D61-Pad2): track 435.4 -> 433.2 mm
- net Net-(D82-Pad2): track 145.5 -> 147.2 mm
- net col1: track 376.6 -> 377.7 mm
- net GND: vias 15 -> 17
Other:
- board text added: "R001 - coseyfannitutti 2019 R002 - lauer2356 2020 (numpad)"
- board text removed: "1"
- board text removed: "coseyfannitutti 2019 - rev1 lauer2356 2020 - rev 2.1 (numpad)"

Commit message: proto feedback incorperated
Parts:
- removed the REF** at (96.4, 161.4)
- removed the REF** at (206.1, 171.0)
- added REF**: MountingHole_2.2mm_M2_Pad, cftkb:MountingHole_2.2mm_M2_Pad, F.Cu at (96.7, 161.4)
- added REF**: MountingHole_2.2mm_M2_Pad, cftkb:MountingHole_2.2mm_M2_Pad, F.Cu at (206.2, 171.0)
Other:
- board text added: "Revised lauer2356 11May2020"
- board text removed: "Revised lauer2356 27April2020"
Changed lines of the file:
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@@
   (general
     (thickness 1.6)
-    (drawings 43)
-    (tracks 2557)
+    (drawings 49)
+    (tracks 2559)
     (zones 0)
     (modules 214)
@@
     (solder_mask_min_width 0.25)
     (aux_axis_origin 63.2142 94.76362)
-    (grid_origin 58.57875 61.43625)
+    (grid_origin 53.8162 180.48862)
     (visible_elements 7FFFFFFF)
     (pcbplotparams
@@
   )
   (module cftkb:MountingHole_2.2mm_M2_Pad (layer F.Cu)
-    (at 206.0892 170.96362)
+    (at 206.21625 170.97375)
     (descr "Mounting Hole 2.2mm, M2")
     (tags "mounting hole 2.2mm m2")
@@
   )
   (module cftkb:MountingHole_2.2mm_M2_Pad (layer F.Cu)
-    (at 96.36125 161.44875)
+    (at 96.67875 161.44875)
     (descr "Mounting Hole 2.2mm, M2")
     (tags "mounting hole 2.2mm m2")
@@
     (descr "Diode, DO-35_SOD27 series, Axial, Horizontal, pin pitch=7.62mm, , length*diameter=4*2mm^2, , http://www.diodes.com/_files/packages/DO-35.pdf")
     (tags "Diode DO-35_SOD27 series Axial Horizontal pin pitch 7.62mm  length 4mm diameter 2mm")
-    (fp_text reference D65 (at 8.77 0 270) (layer F.SilkS)
+    (fp_text reference D65 (at 7.991609 0) (layer F.SilkS)
       (effects (font (size 0.8 0.8) (thickness 0.15)))
     )
@@
     )
   )
-  (gr_text "Revised lauer2356 27April2020" (at 336.6452 201.63412) (layer Cmts.User)
+  (gr_circle (center 63.3412 85.23862) (end 63.3412 87.61987) (layer B.SilkS) (width 0.15))
+  (gr_circle (center 63.3412 173.34487) (end 65.72245 173.34487) (layer B.SilkS) (width 0.15))
+  (gr_circle (center 241.93495 85.23862) (end 241.93495 87.61987) (layer B.SilkS) (width 0.15))
+  (gr_circle (center 241.93495 173.34487) (end 241.93495 175.72612) (layer B.SilkS) (width 0.15))
+  (gr_circle (center 415.7662 85.23862) (end 415.7662 87.61987) (layer B.SilkS) (width 0.15))
+  (gr_circle (center 415.7662 173.34487) (end 415.7662 175.72612) (layer B.SilkS) (width 0.15))
+  (gr_text "Revised lauer2356 11May2020 " (at 336.6452 201.63412) (layer Cmts.User)
     (effects (font (size 1.5 1.5) (thickness 0.3)))
   )
@@
   (segment (start 392.78093 75.257812) (end 390.67517 73.152052) (width 0.25) (layer F.Cu) (net 101))
   (segment (start 392.78093 76.389182) (end 392.78093 75.257812) (width 0.25) (layer F.Cu) (net 101) (status 10))
-  (segment (start 385.737989 79.506241) (end 382.62093 76.389182) (width 0.25) (layer B.Cu) (net 102) (status 20))
-  (segment (start 388.889145 79.506241) (end 385.737989 79.506241) (width 0.25) (layer B.Cu) (net 102))
   (segment (start 389.639144 80.25624) (end 388.889145 79.506241) (width 0.25) (layer B.Cu) (net 102) (status 10))
   (segment (start 391.388944 82.00604) (end 394.293612 82.00604) (width 0.25) (layer B.Cu) (net 102) (status 20))
   (segment (start 389.639144 80.25624) (end 391.388944 82.00604) (width 0.25) (layer B.Cu) (net 102) (status 10))
+  (segment (start 388.889145 79.506241) (end 388.878241 79.506241) (width 0.25) (layer B.Cu) (net 102))
+  (segment (start 388.878241 79.506241) (end 387.06425 77.69225) (width 0.25) (layer B.Cu) (net 102))
+  (segment (start 383.923998 77.69225) (end 382.62093 76.389182) (width 0.25) (layer B.Cu) (net 102))
+  (segment (start 387.06425 77.69225) (end 383.923998 77.69225) (width 0.25) (layer B.Cu) (net 102))
   (segment (start 381.204251 80.186749) (end 380.07925 81.31175) (width 0.25) (layer F.Cu) (net 103) (status 20))
   (segment (start 381.204251 77.512503) (end 381.204251 80.186749) (width 0.25) (layer F.Cu) (net 103))

Commit message: order PCBs and ponoko
Parts:
- removed the REF** at (387.2, 92.4)
- removed the REF** at (301.5, 92.4)
- removed the REF** at (206.2, 94.8)
- removed the REF** at (91.9, 92.4)
- removed the REF** at (244.3, 123.3)
Other:
- board text added: "EL-05/2020"
- board text removed: "R001 - coseyfannitutti 2019 R002 - lauer2356 2020 (numpad)"
Changed lines of the file:
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@@
   (general
     (thickness 1.6)
-    (drawings 49)
+    (drawings 43)
     (tracks 2559)
     (zones 0)
-    (modules 214)
+    (modules 209)
     (nets 128)
   )
@@
   )
   (module cftkb:MountingHole_2.2mm_M2_Pad (layer F.Cu)
-    (at 387.19125 92.3925)
-    (descr "Mounting Hole 2.2mm, M2")
-    (tags "mounting hole 2.2mm m2")
-    (attr virtual)
-    (fp_text reference REF** (at 0 -3.2) (layer Cmts.User)
-      (effects (font (size 1 1) (thickness 0.15)))
-    )
-    (fp_text value MountingHole_2.2mm_M2_Pad (at 0 3.2) (layer F.Fab)
-      (effects (font (size 1 1) (thickness 0.15)))
-    )
-    (fp_text user %R (at 0.3 0) (layer F.Fab)
-      (effects (font (size 1 1) (thickness 0.15)))
-    )
-    (fp_circle (center 0 0) (end 2.2 0) (layer Cmts.User) (width 0.15))
-    (fp_circle (center 0 0) (end 2.45 0) (layer F.CrtYd) (width 0.05))
-    (pad 1 thru_hole circle (at 0 0) (size 4.4 4.4) (drill 2.2) (layers *.Cu *.Mask))
-  )
-  (module cftkb:MountingHole_2.2mm_M2_Pad (layer F.Cu)
-    (at 301.46625 92.3925)
-    (descr "Mounting Hole 2.2mm, M2")
-    (tags "mounting hole 2.2mm m2")
-    (attr virtual)
-    (fp_text reference REF** (at 0 -3.2) (layer Cmts.User)
-      (effects (font (size 1 1) (thickness 0.15)))
-    )
-    (fp_text value MountingHole_2.2mm_M2_Pad (at 0 3.2) (layer F.Fab)
-      (effects (font (size 1 1) (thickness 0.15)))
-    )
-    (fp_text user %R (at 0.3 0) (layer F.Fab)
-      (effects (font (size 1 1) (thickness 0.15)))
-    )
-    (fp_circle (center 0 0) (end 2.2 0) (layer Cmts.User) (width 0.15))
-    (fp_circle (center 0 0) (end 2.45 0) (layer F.CrtYd) (width 0.05))
-    (pad 1 thru_hole circle (at 0 0) (size 4.4 4.4) (drill 2.2) (layers *.Cu *.Mask))
-  )
-  (module cftkb:MountingHole_2.2mm_M2_Pad (layer F.Cu)
-    (at 206.21625 94.77375)
-    (descr "Mounting Hole 2.2mm, M2")
-    (tags "mounting hole 2.2mm m2")
-    (attr virtual)
-    (fp_text reference REF** (at 0 -3.2) (layer Cmts.User)
-      (effects (font (size 1 1) (thickness 0.15)))
-    )
-    (fp_text value MountingHole_2.2mm_M2_Pad (at 0 3.2) (layer F.Fab)
-      (effects (font (size 1 1) (thickness 0.15)))
-    )
-    (fp_text user %R (at 0.3 0) (layer F.Fab)
-      (effects (font (size 1 1) (thickness 0.15)))
-    )
-    (fp_circle (center 0 0) (end 2.2 0) (layer Cmts.User) (width 0.15))
-    (fp_circle (center 0 0) (end 2.45 0) (layer F.CrtYd) (width 0.05))
-    (pad 1 thru_hole circle (at 0 0) (size 4.4 4.4) (drill 2.2) (layers *.Cu *.Mask))
-  )
-  (module cftkb:MountingHole_2.2mm_M2_Pad (layer F.Cu)
-    (at 91.91625 92.3925)
-    (descr "Mounting Hole 2.2mm, M2")
-    (tags "mounting hole 2.2mm m2")
-    (attr virtual)
-    (fp_text reference REF** (at 0 -3.2) (layer Cmts.User)
-      (effects (font (size 1 1) (thickness 0.15)))
-    )
-    (fp_text value MountingHole_2.2mm_M2_Pad (at 0 3.2) (layer F.Fab)
-      (effects (font (size 1 1) (thickness 0.15)))
-    )
-    (fp_text user %R (at 0.3 0) (layer F.Fab)
-      (effects (font (size 1 1) (thickness 0.15)))
-    )
-    (fp_circle (center 0 0) (end 2.2 0) (layer Cmts.User) (width 0.15))
-    (fp_circle (center 0 0) (end 2.45 0) (layer F.CrtYd) (width 0.05))
-    (pad 1 thru_hole circle (at 0 0) (size 4.4 4.4) (drill 2.2) (layers *.Cu *.Mask))
-  )
-  (module cftkb:MountingHole_2.2mm_M2_Pad (layer F.Cu)
     (at 242.41075 61.43625)
     (descr "Mounting Hole 2.2mm, M2")
@@
     )
   )
-  (module cftkb:NumDiscipline_LARGE_B_SILK (layer F.Cu)
-    (at 244.31625 123.34875)
-    (fp_text reference REF** (at 0 5.08) (layer Cmts.User) hide
-      (effects (font (size 1 1) (thickness 0.15)))
-    )
-    (fp_text value NumDiscipline_LARGE_B_SILK (at 0 -0.5) (layer F.Fab)
-      (effects (font (size 1 1) (thickness 0.15)))
-    )
-    (fp_line (start -53.34 15.24) (end 55.88 15.24) (layer B.SilkS) (width 1))
-    (fp_line (start 55.88 -15.24) (end -53.34 -15.24) (layer B.SilkS) (width 1))
-    (fp_arc (start -53.34 0) (end -53.34 -15.24) (angle -180) (layer B.SilkS) (width 1))
-    (fp_arc (start 55.88 0) (end 55.88 15.24) (angle -180) (layer B.SilkS) (width 1))
-    (fp_text user "#Discipline" (at 0 0) (layer B.SilkS)
-      (effects (font (size 15 15) (thickness 2.5)) (justify mirror))
-    )
-  )
   (module cftkb:NumDiscipline_SMALL_COPPER (layer F.Cu)
     (at 152.876 164.49675)
@@
     )
   )
-  (gr_circle (center 63.3412 85.23862) (end 63.3412 87.61987) (layer B.SilkS) (width 0.15))
-  (gr_circle (center 63.3412 173.34487) (end 65.72245 173.34487) (layer B.SilkS) (width 0.15))
-  (gr_circle (center 241.93495 85.23862) (end 241.93495 87.61987) (layer B.SilkS) (width 0.15))
-  (gr_circle (center 241.93495 173.34487) (end 241.93495 175.72612) (layer B.SilkS) (width 0.15))
-  (gr_circle (center 415.7662 85.23862) (end 415.7662 87.61987) (layer B.SilkS) (width 0.15))
-  (gr_circle (center 415.7662 173.34487) (end 415.7662 175.72612) (layer B.SilkS) (width 0.15))
   (gr_text "Revised lauer2356 11May2020 " (at 336.6452 201.63412) (layer Cmts.User)
     (effects (font (size 1.5 1.5) (thickness 0.3)))
@@
     (effects (font (size 1 1) (thickness 0.1)))
   )
-  (gr_text "R001 - coseyfannitutti 2019\nR002 - lauer2356 2020 (numpad)" (at 166.846 172.11675) (layer F.SilkS)
+  (gr_text EL-05/2020 (at 158.5912 178.10737) (layer F.SilkS)
     (effects (font (size 2 1.5) (thickness 0.075)) (justify right))
   )
