File: FR4Plate/FR4Plate.kicad_pcb (KiCad board)
At the start: 2 copper layers, 371.5 x 100.6 mm, 3 parts

Commit message: add 3d, finish plate
Parts:
- moved ... 64.1 mm to (34.6, 125.0)
- moved REF** 64.1 mm to (182.2, 153.5) (x2)
Other:
- outline, holes or cut-outs redrawn

Commit message: start making adjustments from first proto
Parts:
- removed ...: R, Resistor_THT:R_Axial_DIN0204_L3.6mm_D1.6mm_P1.90mm_Vertical
- removed the REF** at (182.2, 153.5) (x2)
- added ?: , , F.Cu at (127.4, 48.8)
- added REF**: MountingHole_3.5mm, MountingHole:MountingHole_3.5mm, F.Cu at (272.7, 144.0)
- added REF**: NumDiscipline_SMALL_FSILK, cftkb:NumDiscipline_SMALL_FSILK, F.Cu at (125.1, 153.5)
- added REF**: MountingHole_3.5mm, MountingHole:MountingHole_3.5mm, F.Cu at (177.5, 144.0)
- added REF**: MountingHole_3.5mm, MountingHole:MountingHole_3.5mm, F.Cu at (358.4, 144.0)
- added REF**: MountingHole_3.5mm, MountingHole:MountingHole_3.5mm, F.Cu at (358.4, 86.9)
- added REF**: MountingHole_3.5mm, MountingHole:MountingHole_3.5mm, F.Cu at (67.9, 144.0)
- added REF**: MountingHole_3.5mm, MountingHole:MountingHole_3.5mm, F.Cu at (63.2, 86.9)
- added REF**: MountingHole_3.5mm, MountingHole:MountingHole_3.5mm, F.Cu at (177.5, 86.9)
- added REF**: MountingHole_3.5mm, MountingHole:MountingHole_3.5mm, F.Cu at (272.7, 86.9)

Commit message: proto feedback incorperated
Parts:
- moved REF** 14.3 mm to (258.4, 144.0)
- moved REF** 9.52 mm to (177.5, 153.5)
Changed lines of the file:
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@@
   )
   (module MountingHole:MountingHole_3.5mm (layer F.Cu)
-    (at 272.7005 144.01875)
+    (at 258.413 144.01875)
     (descr "Mounting Hole 3.5mm, no annular")
     (tags "mounting hole 3.5mm no annular")
@@
   )
   (module MountingHole:MountingHole_3.5mm (layer F.Cu)
-    (at 177.4505 144.01875)
+    (at 177.4505 153.54375)
     (descr "Mounting Hole 3.5mm, no annular")
     (tags "mounting hole 3.5mm no annular")

Commit message: order PCBs and ponoko
Routing:
- added copper zone on B.Cu, net (none)
- added copper zone on F.Cu, net (none)
- removed copper zone on B.Cu, net GND
- removed copper zone on F.Cu, net GND
Changed lines of the file:
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@@
     (zones 0)
     (modules 10)
-    (nets 2)
+    (nets 1)
   )
   (page A3)
@@
   )
   (net 0 "")
-  (net 1 GND)
   (net_class Default "This is the default net class."
     (clearance 0.2)
@@
     (uvia_dia 0.3)
     (uvia_drill 0.1)
-    (add_net GND)
   )
   (module MountingHole:MountingHole_3.5mm (layer F.Cu)
@@
     (tags "mounting hole 3.5mm no annular")
     (attr virtual)
-    (fp_text reference REF** (at 0 -4.5) (layer F.SilkS)
+    (fp_text reference REF** (at 0 -4.5) (layer Cmts.User)
       (effects (font (size 1 1) (thickness 0.15)))
     )
@@
     (tags "mounting hole 3.5mm no annular")
     (attr virtual)
-    (fp_text reference REF** (at 0 -4.5) (layer F.SilkS)
+    (fp_text reference REF** (at 0 -4.5) (layer Cmts.User)
       (effects (font (size 1 1) (thickness 0.15)))
     )
@@
     (tags "mounting hole 3.5mm no annular")
     (attr virtual)
-    (fp_text reference REF** (at 0 -4.5) (layer F.SilkS)
+    (fp_text reference REF** (at 0 -4.5) (layer Cmts.User)
       (effects (font (size 1 1) (thickness 0.15)))
     )
@@
     (tags "mounting hole 3.5mm no annular")
     (attr virtual)
-    (fp_text reference REF** (at 0 -4.5) (layer F.SilkS)
+    (fp_text reference REF** (at 0 -4.5) (layer B.Fab)
       (effects (font (size 1 1) (thickness 0.15)))
     )
@@
     (tags "mounting hole 3.5mm no annular")
     (attr virtual)
-    (fp_text reference REF** (at 0 -4.5) (layer F.SilkS)
+    (fp_text reference REF** (at 0 -4.5) (layer Cmts.User)
       (effects (font (size 1 1) (thickness 0.15)))
     )
@@
     (tags "mounting hole 3.5mm no annular")
     (attr virtual)
-    (fp_text reference REF** (at 0 -4.5) (layer F.SilkS)
+    (fp_text reference REF** (at 0 -4.5) (layer Cmts.User)
       (effects (font (size 1 1) (thickness 0.15)))
     )
@@
     (tags "mounting hole 3.5mm no annular")
     (attr virtual)
-    (fp_text reference REF** (at 0 -4.5) (layer F.SilkS)
+    (fp_text reference REF** (at 0 -4.5) (layer Cmts.User)
       (effects (font (size 1 1) (thickness 0.15)))
     )
@@
     (tags "mounting hole 3.5mm no annular")
     (attr virtual)
-    (fp_text reference REF** (at 0 -4.5) (layer F.SilkS)
+    (fp_text reference REF** (at 0 -4.5) (layer Cmts.User)
       (effects (font (size 1 1) (thickness 0.15)))
     )
@@
   (gr_arc (start 323.8505 128.49375) (end 323.8505 127.49375) (angle -90) (layer Edge.Cuts) (width 0.05))
   (gr_arc (start 323.8505 140.49375) (end 322.8505 140.49375) (angle -90) (layer Edge.Cuts) (width 0.05))
-  (zone (net 1) (net_name GND) (layer F.Cu) (hatch edge 0.508)
+  (zone (net 0) (net_name "") (layer F.Cu) (hatch edge 0.508)
     (connect_pads (clearance 0.508))
     (min_thickness 0.254)
@@
     )
   )
-  (zone (net 1) (net_name GND) (layer B.Cu) (hatch edge 0.508)
+  (zone (net 0) (net_name "") (layer B.Cu) (hatch edge 0.508)
     (connect_pads (clearance 0.508))
     (min_thickness 0.254)
